File: HARDWARE/KICAD/mini_futbolista.kicad_sch (KiCad schematic)
At the start: 5 parts, among them J1 Screw_Terminal_01x02, J2 Screw_Terminal_01x02, U1 ESP32-C3_SUPERMINI_TH

Commit message: revisado
Parts:
- added C1, C2: C_Polarized, Capacitor_THT:CP_Radial_D8.0mm_P5.00mm, symbol Device:C_Polarized
- added C3, C4: C, Capacitor_THT:C_Disc_D5.0mm_W2.5mm_P2.50mm, symbol Device:C
- added J3: ENTRADA BATERIA, TerminalBlock:TerminalBlock_MaiXu_MX126-5.0-02P_1x02_P5.00mm, symbol Connector:Screw_Terminal_01x02
- added J4: LLAVE ENCENDIDO, TerminalBlock:TerminalBlock_MaiXu_MX126-5.0-02P_1x02_P5.00mm, symbol Connector:Screw_Terminal_01x02
- added J5: Conn_01x04_Pin, Connector_PinHeader_2.54mm:PinHeader_1x04_P2.54mm_Vertical, symbol Connector:Conn_01x04_Pin
Connections:
- net +5V: now also U2.3 (OUT_+), C2.1, J5.4 (Pin_4)
- net AIN1: now also U1.5 (GPIO5); no longer U1.4 (GPIO4)
- net AIN2: now also U1.3 (GPIO3); no longer U1.5 (GPIO5)
- net BIN1: now also U1.7 (GPIO7); no longer U1.6 (GPIO6)
- net BIN2: now also U1.4 (GPIO4); no longer U1.7 (GPIO7)
- net ECHO: now also U1.20 (GPIO20), J5.2 (Pin_2); no longer U1.9 (GPIO9)
- net GND: now also U2.1 (-IN), U2.4 (OUT_-), C1.2, C2.2, J3.1 (Pin_1), J5.1 (Pin_1)
- net OUT1: now also C3.1
- net OUT2: now also C3.2
- net OUT3: now also C4.1
- net OUT4: now also C4.2
- net TRIG: now also U1.10 (GPIO10), J5.3 (Pin_3); no longer U1.8 (GPIO8)
- net VCC: now also J3.2 (Pin_2), J4.1 (Pin_1)
- new net: C1.1, J4.2 (Pin_2), U2.2 (+IN)
Other:
- moved on the sheet: J1
