File: HARDWARE/KICAD/mini_futbolista.kicad_pcb (KiCad board)
At the start: 2 copper layers, 99.5 x 49.5 mm, 5 parts, among them J1 Screw_Terminal_01x02, J2 Screw_Terminal_01x02, U1 ESP32-C3_SUPERMINI_TH

Commit message: revisado
Parts:
- added C1: C_Polarized, Capacitor_THT:CP_Radial_D8.0mm_P5.00mm, F.Cu at (177.1, 100.5)
- added C2: C_Polarized, Capacitor_THT:CP_Radial_D8.0mm_P5.00mm, F.Cu at (177.6, 68.0)
- added C3: C, Capacitor_THT:C_Disc_D5.0mm_W2.5mm_P2.50mm, F.Cu at (199.0, 67.0)
- added C4: C, Capacitor_THT:C_Disc_D5.0mm_W2.5mm_P2.50mm, F.Cu at (147.5, 66.5)
- added G***: LOGO, VARIOS:LOGO_EESTN5_F.Cu, B.Cu at (202.5, 101.5)
- added J3: ENTRADA BATERIA, TerminalBlock:TerminalBlock_MaiXu_MX126-5.0-02P_1x02_P5.00mm, F.Cu at (192.0, 104.5)
- added J4: LLAVE ENCENDIDO, TerminalBlock:TerminalBlock_MaiXu_MX126-5.0-02P_1x02_P5.00mm, F.Cu at (172.5, 105.0)
- added J5: Conn_01x04_Pin, Connector_PinHeader_2.54mm:PinHeader_1x04_P2.54mm_Vertical, F.Cu at (158.9, 98.0)
- moved U2 35.6 mm to (145.2, 94.0), turned to 90 degrees
- moved DRV1 3.77 mm to (188.1, 84.5)
- moved U1 2.00 mm to (167.5, 83.0)
Connections:
- U1 pad 10: unconnected-(U1-GPIO10-Pad10) -> TRIG
- U1 pad 20: unconnected-(U1-GPIO20-Pad20) -> ECHO
- U1 pad 3: unconnected-(U1-GPIO3-Pad3) -> AIN2
- U1 pad 4: AIN1 -> BIN2
- U1 pad 5: AIN2 -> AIN1
- U1 pad 6: BIN1 -> unconnected-(U1-GPIO6-Pad6)
- U1 pad 7: BIN2 -> BIN1
- U1 pad 8: TRIG -> unconnected-(U1-GPIO8-Pad8)
- U1 pad 9: ECHO -> unconnected-(U1-GPIO9-Pad9)
- U2 pad 1: (no net) -> GND
- U2 pad 2: (no net) -> Net-(J4-Pin_2)
- U2 pad 3: (no net) -> +5V
- U2 pad 4: (no net) -> GND
Routing:
- net +5V: track 0.00 -> 76.1 mm
- net BIN2: track 64.0 -> 24.6 mm
- net AIN2: track 51.5 -> 21.1 mm
- net VCC: track 0.00 -> 30.1 mm
- net AIN1: track 14.7 -> 41.1 mm
- net Net-(J4-Pin_2): track 0.00 -> 25.8 mm
- net OUT1: track 16.2 -> 33.1 mm
- net TRIG: track 0.00 -> 16.9 mm
- net GND: track 27.9 -> 14.5 mm
- net ECHO: track 0.00 -> 12.6 mm
- net OUT2: track 28.6 -> 36.4 mm
- net BIN1: track 49.3 -> 43.2 mm
- net OUT4: track 54.1 -> 58.9 mm
- net OUT3: track 57.2 -> 62.0 mm
- added copper zone on B.Cu, net GND

Commit message: con pdf
Parts:
- added C1: C_Polarized, Capacitor_THT:CP_Radial_D8.0mm_P5.00mm, F.Cu at (225.5, 106.9)
- added C2: C_Polarized, Capacitor_THT:CP_Radial_D8.0mm_P5.00mm, F.Cu at (193.0, 106.4)
- added C3: C, Capacitor_THT:C_Disc_D5.0mm_W2.5mm_P2.50mm, F.Cu at (192.0, 85.0)
- added C4: C, Capacitor_THT:C_Disc_D5.0mm_W2.5mm_P2.50mm, F.Cu at (191.5, 136.5)
- added DRV1: PUENTE H, DRV8833:DRV8833, F.Cu at (209.5, 95.9)
- added G***: LOGO, VARIOS:LOGO_EESTN5_F.Cu, B.Cu at (226.5, 81.5)
- added J1: Screw_Terminal_01x02, TerminalBlock:TerminalBlock_MaiXu_MX126-5.0-02P_1x02_P5.00mm, F.Cu at (197.0, 139.5)
- added J2: Screw_Terminal_01x02, TerminalBlock:TerminalBlock_MaiXu_MX126-5.0-02P_1x02_P5.00mm, F.Cu at (202.0, 78.5)
- added J3: ENTRADA BATERIA, TerminalBlock:TerminalBlock_MaiXu_MX126-5.0-02P_1x02_P5.00mm, F.Cu at (229.5, 92.0)
- added J4: LLAVE ENCENDIDO, TerminalBlock:TerminalBlock_MaiXu_MX126-5.0-02P_1x02_P5.00mm, F.Cu at (230.0, 111.5)
- added J5: Conn_01x04_Pin, Connector_PinHeader_2.54mm:PinHeader_1x04_P2.54mm_Vertical, F.Cu at (223.0, 125.1)
- added U1: ESP32-C3_SUPERMINI_TH, ESP32-C3_SUPERMINI_TH:MODULE_ESP32-C3_SUPERMINI, F.Cu at (208.0, 116.5)
- added U2: ~, mini360:mini360, F.Cu at (219.0, 138.8)
- moved C3 147.1 mm to (53.0, 85.0), turned to 90 degrees
- moved J2 142.5 mm to (63.0, 78.5), turned to 180 degrees
- moved C2 129.4 mm to (54.0, 106.4), turned to 90 degrees
- moved DRV1 118.1 mm to (70.5, 95.9), turned to 0 degrees
- moved C4 118.0 mm to (52.5, 136.5), turned to 90 degrees
- moved G*** 116.7 mm to (87.5, 81.5), turned to -90 degrees
- moved J1 109.7 mm to (58.0, 139.5), turned to 0 degrees
- moved U1 104.0 mm to (69.0, 116.5), turned to 90 degrees
- moved J3 102.2 mm to (90.5, 92.0), turned to -90 degrees
- moved C1 90.8 mm to (86.5, 106.9), turned to 90 degrees
- moved J4 81.8 mm to (91.0, 111.5), turned to -90 degrees
- moved J5 79.7 mm to (84.0, 125.1), turned to 180 degrees
- moved U2 79.2 mm to (80.0, 138.8), turned to 180 degrees
Routing:
- net +5V: track 76.1 -> 152.2 mm
- net OUT3: track 62.0 -> 123.9 mm
- net OUT4: track 58.9 -> 117.8 mm
- net BIN1: track 43.2 -> 86.4 mm
- net AIN1: track 41.1 -> 82.3 mm
- net OUT2: track 36.4 -> 72.8 mm
- net OUT1: track 33.1 -> 66.2 mm
- net VCC: track 30.1 -> 60.1 mm
- net Net-(J4-Pin_2): track 25.8 -> 51.7 mm
- net BIN2: track 24.6 -> 49.3 mm
- net AIN2: track 21.1 -> 42.1 mm
- net TRIG: track 16.9 -> 33.8 mm
- net GND: track 14.5 -> 28.9 mm
- net ECHO: track 12.6 -> 25.2 mm
Other:
- board size 99.5 x 49.5 mm -> 188.5 x 99.5 mm
